File: 12-volts-dimmer.kicad_sch (KiCad schematic)
At the start: 19 parts, among them IC1 NE556, K1 + L G G, P1 1M, T1 MCU80N03A

Commit message: Minor updates.
Parts:
- C4: Mouser Part Number 0-C0603C103J5RAC -> 80-C0603C103J5RAC
- L1: Mouser Part Number 652-SRU1048-3R0Y -> 652-SRU1048-3R0Y
Changed lines of the file:
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@@
       (effects (font (size 1.27 1.27)) hide)
     )
-    (property "Mouser Part Number" " 652-SRU1048-3R0Y" (id 4) (at 209.55 89.535 0)
+    (property "Mouser Part Number" "652-SRU1048-3R0Y" (id 4) (at 209.55 89.535 0)
       (effects (font (size 1.27 1.27)) hide)
     )
@@
       (effects (font (size 1.27 1.27)) hide)
     )
-    (property "Mouser Part Number" "0-C0603C103J5RAC" (id 4) (at 170.18 88.9 0)
+    (property "Mouser Part Number" "80-C0603C103J5RAC" (id 4) (at 170.18 88.9 0)
       (effects (font (size 1.27 1.27)) hide)
     )
